Commit message: sensors working in both sim and hardware... added sensor relays

File: robot.urdf.xacro (robot description, xacro)
@@ -24,16 +24,16 @@
   <!-- lidar3d_0 -->
   <xacro:include filename="$(find clearpath_sensors_description)/urdf/ouster_os1.urdf.xacro"/>
-  <xacro:ouster_os1 name="lidar3d_0" parent_link="default_mount" min_ang_h="-3.141592" max_ang_h="3.141592" min_ang_v="-0.261799" max_ang_v="0.261799" min_range="0.9" max_range="130.0" update_rate="20" samples_h="1024" samples_v="64" base="base" cap="halo">
-    <origin xyz="0.0 0.0 0.0" rpy="0.0 0.0 0.0"/>
+  <xacro:ouster_os1 name="lidar3d_0" parent_link="default_mount" min_ang_h="-3.141592" max_ang_h="3.141592" min_ang_v="-0.261799" max_ang_v="0.261799" min_range="0.9" max_range="130.0" update_rate="20" samples_h="1024" samples_v="64" base="none" cap="fins">
+    <origin xyz="0.213 0.0 0.2" rpy="0.0 0.0 0.0"/>
   </xacro:ouster_os1>
   <!-- imu_0 -->
   <xacro:include filename="$(find clearpath_sensors_description)/urdf/microstrain_imu.urdf.xacro"/>
   <xacro:microstrain_imu name="imu_0" parent_link="default_mount" update_rate="100">
-    <origin xyz="0.0 0.0 0.0" rpy="0.0 0.0 0.0"/>
+    <origin xyz="0.215 0.102 0.11" rpy="0.0 0.0 0.0"/>
   </xacro:microstrain_imu>
   <!-- gps_0 -->
   <xacro:include filename="$(find clearpath_sensors_description)/urdf/swiftnav_duro.urdf.xacro"/>
   <xacro:swiftnav_duro name="gps_0" parent_link="default_mount">
-    <origin xyz="0.0 0.0 0.0" rpy="0.0 0.0 0.0"/>
+    <origin xyz="0.215 0.0 0.29" rpy="0.0 0.0 0.0"/>
   </xacro:swiftnav_duro>
   <!-- Manipulators -->
